File: led_array/led_array.kicad_pcb (KiCad board)
At the start: 2 copper layers, 39.6 x 30.5 mm, 11 parts

Commit message: update pcb
Parts:
- added MH1: MountingHole, led_array:MountingHole_0-80, F.Cu at (123.4, 113.8)
- added MH2: MountingHole, led_array:MountingHole_0-80, F.Cu at (123.4, 100.3)
- added MH3: MountingHole, led_array:MountingHole_0-80, F.Cu at (160.0, 100.3)
- added MH4: MountingHole, led_array:MountingHole_0-80, F.Cu at (160.0, 113.7)
- renumbered GREEN3 to GREEN1, RED3 to RED1, RED3 to RED2
Connections:
- U$1 pad 1: /FLOAT -> (no net)
- U$2 pad 2: /SIG -> (no net)
Changed lines of the file:
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@@
     (tracks 55)
     (zones 0)
-    (modules 11)
-    (nets 8)
+    (modules 15)
+    (nets 6)
   )
   (page A)
@@
     (mod_text_size 1 1)
     (mod_text_width 0.15)
-    (pad_size 1.016 1.016)
-    (pad_drill 0.508)
+    (pad_size 1.27 1.27)
+    (pad_drill 1.27)
     (pad_to_mask_clearance 0.2)
     (aux_axis_origin 121.92 121.92)
@@
       (outputformat 1)
       (mirror false)
-      (drillshape 1)
+      (drillshape 0)
       (scaleselection 1)
       (outputdirectory ""))
@@
   (net 3 "Net-(GREEN1-PadC)")
   (net 4 /GND)
-  (net 5 /FLOAT)
-  (net 6 /BATT)
-  (net 7 /SIG)
+  (net 5 /BATT)
   (net_class Default "This is the default net class."
     (clearance 0.2)
@@
     (uvia_drill 0.1)
     (add_net /BATT)
-    (add_net /FLOAT)
     (add_net /GND)
-    (add_net /SIG)
     (add_net /VCC)
     (add_net "Net-(GREEN1-PadC)")
     (add_net "Net-(R1-Pad1)")
+  )
+  (module led_array:MountingHole_0-80 (layer Top)
+    (at 160.02 113.665)
+    (descr "Mounting Hole 2.2mm, no annular, M2")
+    (tags "mounting hole 2.2mm no annular m2")
+    (fp_text reference MH4 (at 0 -3.2) (layer F.SilkS) hide
+      (effects (font (size 1 1) (thickness 0.15)))
+    )
+    (fp_text value MountingHole (at 0 3.2) (layer F.Fab)
+      (effects (font (size 1 1) (thickness 0.15)))
+    )
+    (fp_circle (center 0 0) (end 1.6 0) (layer F.CrtYd) (width 0.05))
+    (fp_circle (center 0 0) (end 1.6 0) (layer Cmts.User) (width 0.15))
+    (pad "" np_thru_hole circle (at 0 0) (size 1.27 1.27) (drill 1.27) (layers *.Cu *.Mask))
+  )
+  (module led_array:MountingHole_0-80 (layer Top)
+    (at 160.02 100.33)
+    (descr "Mounting Hole 2.2mm, no annular, M2")
+    (tags "mounting hole 2.2mm no annular m2")
+    (fp_text reference MH3 (at 0 -3.2) (layer F.SilkS) hide
+      (effects (font (size 1 1) (thickness 0.15)))
+    )
+    (fp_text value MountingHole (at 0 3.2) (layer F.Fab)
+      (effects (font (size 1 1) (thickness 0.15)))
+    )
+    (fp_circle (center 0 0) (end 1.6 0) (layer Cmts.User) (width 0.15))
+    (fp_circle (center 0 0) (end 1.6 0) (layer F.CrtYd) (width 0.05))
+    (pad "" np_thru_hole circle (at 0 0) (size 1.27 1.27) (drill 1.27) (layers *.Cu *.Mask))
+  )
+  (module led_array:MountingHole_0-80 (layer Top)
+    (at 123.444 100.33)
+    (descr "Mounting Hole 2.2mm, no annular, M2")
+    (tags "mounting hole 2.2mm no annular m2")
+    (fp_text reference MH2 (at 0 -3.2) (layer F.SilkS) hide
+      (effects (font (size 1 1) (thickness 0.15)))
+    )
+    (fp_text value MountingHole (at 0 3.2) (layer F.Fab)
+      (effects (font (size 1 1) (thickness 0.15)))
+    )
+    (fp_circle (center 0 0) (end 1.6 0) (layer F.CrtYd) (width 0.05))
+    (fp_circle (center 0 0) (end 1.6 0) (layer Cmts.User) (width 0.15))
+    (pad "" np_thru_hole circle (at 0 0) (size 1.27 1.27) (drill 1.27) (layers *.Cu *.Mask))
+  )
+  (module led_array:MountingHole_0-80 (layer Top)
+    (at 123.444 113.792)
+    (descr "Mounting Hole 2.2mm, no annular, M2")
+    (tags "mounting hole 2.2mm no annular m2")
+    (fp_text reference MH1 (at 0 -3.2) (layer F.SilkS) hide
+      (effects (font (size 1 1) (thickness 0.15)))
+    )
+    (fp_text value MountingHole (at 0 3.2) (layer F.Fab)
+      (effects (font (size 1 1) (thickness 0.15)))
+    )
+    (fp_circle (center 0 0) (end 1.6 0) (layer Cmts.User) (width 0.15))
+    (fp_circle (center 0 0) (end 1.6 0) (layer F.CrtYd) (width 0.05))
+    (pad "" np_thru_hole circle (at 0 0) (size 1.27 1.27) (drill 1.27) (layers *.Cu *.Mask))
   )
   (module led_array:LED_SML0603 (layer Top)
@@
     (at 123.444 106.68 90)
     (descr "<b>SML0603-XXX (HIGH INTENSITY) LED</b><p>\n<table>\n<tr><td>AG3K</td><td>AQUA GREEN</td></tr>\n<tr><td>B1K</td><td>SUPER BLUE</td></tr>\n<tr><td>R1K</td><td>SUPER RED</td></tr>\n<tr><td>R3K</td><td>ULTRA RED</td></tr>\n<tr><td>O3K</td><td>SUPER ORANGE</td></tr>\n<tr><td>O3KH</td><td>SOFT ORANGE</td></tr>\n<tr><td>Y3KH</td><td>SUPER YELLOW</td></tr>\n<tr><td>Y3K</td><td>SUPER YELLOW</td></tr>\n<tr><td>2CW</td><td>WHITE</td></tr>\n</table>\nSource: http://www.ledtronics.com/ds/smd-0603/Dstr0092.pdf")
-    (fp_text reference RED3 (at -1 -1 90) (layer F.SilkS) hide
+    (fp_text reference RED2 (at -1 -1 90) (layer F.SilkS) hide
       (effects (font (size 1.2065 1.2065) (thickness 0.1016)) (justify left bottom))
     )
@@
       (net 2 /VCC) (solder_mask_margin 0.1016))
     (pad 2 smd rect (at -4.3 0 90) (size 2.5 1) (layers Top F.Paste F.Mask)
-      (net 6 /BATT) (solder_mask_margin 0.1016))
+      (net 5 /BATT) (solder_mask_margin 0.1016))
     (pad 1 smd rect (at -4.3 -1.5 90) (size 2.5 1) (layers Top F.Paste F.Mask)
-      (net 5 /FLOAT) (solder_mask_margin 0.1016))
+      (solder_mask_margin 0.1016))
   )
   (module led_array:LED_SML0603 (layer Top)
     (at 123.444 119.888 90)
     (descr "<b>SML0603-XXX (HIGH INTENSITY) LED</b><p>\n<table>\n<tr><td>AG3K</td><td>AQUA GREEN</td></tr>\n<tr><td>B1K</td><td>SUPER BLUE</td></tr>\n<tr><td>R1K</td><td>SUPER RED</td></tr>\n<tr><td>R3K</td><td>ULTRA RED</td></tr>\n<tr><td>O3K</td><td>SUPER ORANGE</td></tr>\n<tr><td>O3KH</td><td>SOFT ORANGE</td></tr>\n<tr><td>Y3KH</td><td>SUPER YELLOW</td></tr>\n<tr><td>Y3K</td><td>SUPER YELLOW</td></tr>\n<tr><td>2CW</td><td>WHITE</td></tr>\n</table>\nSource: http://www.ledtronics.com/ds/smd-0603/Dstr0092.pdf")
-    (fp_text reference RED3 (at -1 -1 90) (layer F.SilkS) hide
+    (fp_text reference RED1 (at -1 -1 90) (layer F.SilkS) hide
       (effects (font (size 1.2065 1.2065) (thickness 0.1016)) (justify left bottom))
     )
@@
     (at 160.02 119.888 90)
     (descr "<b>SML0603-XXX (HIGH INTENSITY) LED</b><p>\n<table>\n<tr><td>AG3K</td><td>AQUA GREEN</td></tr>\n<tr><td>B1K</td><td>SUPER BLUE</td></tr>\n<tr><td>R1K</td><td>SUPER RED</td></tr>\n<tr><td>R3K</td><td>ULTRA RED</td></tr>\n<tr><td>O3K</td><td>SUPER ORANGE</td></tr>\n<tr><td>O3KH</td><td>SOFT ORANGE</td></tr>\n<tr><td>Y3KH</td><td>SUPER YELLOW</td></tr>\n<tr><td>Y3K</td><td>SUPER YELLOW</td></tr>\n<tr><td>2CW</td><td>WHITE</td></tr>\n</table>\nSource: http://www.ledtronics.com/ds/smd-0603/Dstr0092.pdf")
-    (fp_text reference GREEN3 (at -1 -1 90) (layer F.SilkS) hide
+    (fp_text reference GREEN1 (at -1 -1 90) (layer F.SilkS) hide
       (effects (font (size 1.2065 1.2065) (thickness 0.1016)) (justify left bottom))
     )
@@
       (net 2 /VCC) (solder_mask_margin 0.1016))
     (pad 2 thru_hole circle (at -0.0762 0 270) (size 1.016 1.016) (drill 0.508) (layers *.Cu *.Mask)
-      (net 7 /SIG) (solder_mask_margin 0.1016))
+      (solder_mask_margin 0.1016))
   )
   (module led_array:JST_CONN_HEADER_PH_TOP_2POS_2MM (layer Top)
@@
     (fp_line (start -2.95 -1.7) (end 2.95 -1.7) (layer F.SilkS) (width 0.127))
     (pad PWR thru_hole circle (at -1 0) (size 1.208 1.208) (drill 0.7) (layers *.Cu *.Mask)
-      (net 6 /BATT) (solder_mask_margin 0.1016))
+      (net 5 /BATT) (solder_mask_margin 0.1016))
     (pad GND thru_hole circle (at 1 0) (size 1.208 1.208) (drill 0.7) (layers *.Cu *.Mask)
       (net 4 /GND) (solder_mask_margin 0.1016))
@@
     (effects (font (size 1.27 1.5) (thickness 0.2032)))
   )
-  (gr_text GREEN (at 160.02 113.284 90) (layer F.SilkS)
+  (gr_text GREEN (at 154.94 92.71) (layer F.SilkS)
     (effects (font (size 1.27 1.5) (thickness 0.2032)))
   )
-  (gr_text RED (at 123.444 113.284 90) (layer F.SilkS)
+  (gr_text RED (at 127 92.71) (layer F.SilkS)
     (effects (font (size 1.27 1.5) (thickness 0.2032)))
   )
@@
   (via (at 134.62 120.396) (size 0.8) (drill 0.4) (layers Top Bottom) (net 4))
   (via (at 139.7 120.396) (size 0.8) (drill 0.4) (layers Top Bottom) (net 4))
-  (segment (start 146.828 111.252) (end 146.812 111.252) (width 0.508) (layer Top) (net 6))
-  (segment (start 146.812 111.252) (end 146.304 110.744) (width 0.508) (layer Top) (net 6))
-  (segment (start 146.304 110.744) (end 141.224 110.744) (width 0.508) (layer Top) (net 6))
-  (segment (start 137.16 114.808) (end 137.16 116.604) (width 0.508) (layer Top) (net 6))
-  (segment (start 141.224 110.744) (end 137.16 114.808) (width 0.508) (layer Top) (net 6))
+  (segment (start 146.828 111.252) (end 146.812 111.252) (width 0.508) (layer Top) (net 5))
+  (segment (start 146.812 111.252) (end 146.304 110.744) (width 0.508) (layer Top) (net 5))
+  (segment (start 146.304 110.744) (end 141.224 110.744) (width 0.508) (layer Top) (net 5))
+  (segment (start 137.16 114.808) (end 137.16 116.604) (width 0.508) (layer Top) (net 5))
+  (segment (start 141.224 110.744) (end 137.16 114.808) (width 0.508) (layer Top) (net 5))
   (zone (net 4) (net_name /GND) (layer Bottom) (hatch edge 0.508)
     (priority 6)
